File: experiments/seven_segment/seven_segment.kicad_sch (KiCad schematic)
At the start: 25 parts, among them J1 Raspberry Pi Pico H, J2 UART0, SW1 Reset, U1 SN74AHC595N, U2 SN74AHC595N, U3 TDSO1160-KL, U4 TDSG1160-LM

Commit message: feat: Finish seven segment experiment
Create prototype driver for chained seven segment displays paired with shift registers.
Parts:
- removed U3: TDSO1160-KL, Display_7Segment:D1X8K, symbol Display_Character:D148K
- removed U4: TDSG1160-LM, Display_7Segment:D1X8K, symbol Display_Character:D148K
- added U1: MAN6740, Display_7Segment:DA56-11SURKWA, symbol Display_Character:DC56-11EWA
- renumbered C2 to C1, C3 to C2, J2 to J1, J1 to J2, U1 to U2, U2 to U3
Connections:
- net GND: now also U1.13 (DIG2_CC), U1.14 (DIG1_CC)
- net at R14.1: now also U1.12 (DIG2_F)
- net at R11.1: now also U1.8 (DIG2_C)
- net at R7.1: now also U1.17 (DIG1_G)
- net at R9.1: now also U1.11 (DIG2_A)
- net at R4.1: now also U1.2 (DIG1_D)
- net at R10.1: now also U1.10 (DIG2_B)
- net at R15.1: now also U1.7 (DIG2_G)
- net at R8.1: now also U1.4 (DP1)
- net at R3.1: now also U1.3 (DIG1_C)
- net at R1.1: now also U1.16 (DIG1_A)
- net at R5.1: now also U1.1 (DIG1_E)
- net at R12.1: now also U1.6 (DIG2_D)
- net at R2.1: now also U1.15 (DIG1_B)
- net at R13.1: now also U1.5 (DIG2_E)
- net at R16.1: now also U1.9 (DP2)
- net at R6.1: now also U1.18 (DIG1_F)
Other:
- note removed: "High"
- note removed: "Low"
- moved on the sheet: C1, C2, J1, J2, R1, R10, R11, R12, R13, R14, R15, R16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
